File: _autosave-GP22_board.kicad_pcb (KiCad board)
At the start: 2 copper layers, 100 x 100 mm, 115 parts, among them CON1 5V power input, IC1 ATMEGA328P-A, P1 TTLOut1, P10 CONN_02X02, P11 CONN_02X02, P12 CONN_02X02, P13 TTLOut2, P14 TTLOut3, P15 CONN_01X03, P2 SineInput, P3 TTLInput, P4 USB_OTG, P5 ICSP, P6 StraightThroughInput, P7 CONN_02X02, P8 CONN_02X02, P9 CONN_02X02, SW1 ROTARY_SWITCH_ALPS_SRBM, SW2 ROTARY_SWITCH_ALPS_SRBM, SW3 ROTARY_SWITCH_ALPS_SRBM, U1 RS 252-210, U10 XC6206, U11 ISO7242, U12 FT232RL, U2 GP22, U3 LTC6957-4, U4 ISO3088, U5 IDT49FCT, U6 LD1117S33TR, U7 MC74VHC1GT04, U8 SN74LV8154, U9 SC74HC165N, X1 TSX-3225 X1E0000210013, Y1 4MHz, Y2 32.768 kHz

Commit message: Route the signals! And replace the diodes
Parts:
- moved U7 5.06 mm to (233.2, 79.0)
Changed lines of the file:
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@@
   )
   (module TO_SOT_Packages_SMD:SOT-353_SC-70-5_Handsoldering (layer F.Cu)
-    (at 230.5 83.25)
+    (at 233.25 79)
     (descr "SOT-353, SC-70-5, Handsoldering")
     (attr smd)
