File: PCB/DIYino.sch (KiCad schematic (older format))
At the start: 22 parts, among them IC1 ATMEGA328P-A, P4 USB_OTG, P5 ICSP, U11 ISO7242, U12 FT232RL, X1 TSX-3225 X1E0000210013

Commit message: Update sch for new kicad version
Parts:
- IC1: symbol ATMEGA328P-A -> ATMEGA328P-AU
- P5: symbol CONN_02X03 -> Conn_02x03_Counter_Clockwise
Connections:
- wire segments 86 -> 92
- no-connect marks 16 -> 17
Other:
- moved on the sheet: P4
Changed lines of the file:
@@
 EESchema Schematic File Version 2
+LIBS:GP22_board-rescue
 LIBS:power
 LIBS:device
@@
 $EndDescr
 $Comp
-L ATMEGA328P-A IC1
+L ATMEGA328P-AU IC1
 U 1 1 56BA55CF
 P 1900 3900
@@
 L USB_OTG P4
 U 1 1 56BA5671
-P 1050 6700
-F 0 "P4" H 1375 6575 50  0000 C CNN
-F 1 "USB_OTG" H 1050 6900 50  0000 C CNN
-F 2 "Custom:MICRO-B_USB_TOP_MOUNT" V 1000 6600 60  0001 C CNN
-F 3 "" V 1000 6600 60  0000 C CNN
-	1    1050 6700
+P 1200 6825
+F 0 "P4" H 1525 6700 50  0000 C CNN
+F 1 "USB_OTG" V 950 6825 50  0000 C CNN
+F 2 "Custom:MICRO-B_USB_TOP_MOUNT" V 1150 6725 60  0001 C CNN
+F 3 "" V 1150 6725 60  0000 C CNN
+	1    1200 6825
 	0    1    1    0
 $EndComp
-Text Label 750  6500 2    60   ~ 0
+Text Label 1375 7325 3    60   ~ 0
 USB_5V
-NoConn ~ 750  6800
 NoConn ~ 7250 2750
 NoConn ~ 7250 2900
@@
 5V
 $Comp
-L CONN_02X03 P5
+L Conn_02x03_Counter_Clockwise P5
 U 1 1 56BA568C
-P 2400 6750
-F 0 "P5" H 2400 6950 50  0000 C CNN
-F 1 "ICSP" H 2400 6550 50  0000 C CNN
-F 2 "Pin_Headers:Pin_Header_Straight_2x03" H 2400 5550 60  0001 C CNN
-F 3 "" H 2400 5550 60  0000 C CNN
-	1    2400 6750
+P 2350 6750
+F 0 "P5" H 2350 6950 50  0000 C CNN
+F 1 "ICSP" H 2350 6550 50  0000 C CNN
+F 2 "Pin_Headers:Pin_Header_Straight_2x03" H 2350 5550 60  0001 C CNN
+F 3 "" H 2350 5550 60  0000 C CNN
+	1    2350 6750
 	1    0    0    -1
 $EndComp
@@
 Text Label 9450 3050 0    60   ~ 0
 USB_D+
-Text Label 750  6700 2    60   ~ 0
+Text Label 1200 7125 3    60   ~ 0
 USB_D+
-Text Label 750  6600 2    60   ~ 0
+Text Label 1100 7125 3    60   ~ 0
 USB_D-
 Text Notes 450  6100 0    60   ~ 0
@@
 Text Label 4200 5850 3    60   ~ 0
 GND
-Text Label 1150 7300 3    60   ~ 0
+Text Label 650  6800 1    60   ~ 0
 USB_GND
 Text Label 9450 4450 3    60   ~ 0
@@
 Connection ~ 8500 4750
 Wire Wire Line
-	1150 7100 1150 7300
-Wire Wire Line
-	1150 7150 750  7150
-Wire Wire Line
-	750  7150 750  6900
-Connection ~ 1150 7150
-Wire Wire Line
 	2650 6850 2650 7000
 Wire Wire Line
 	2650 6500 2650 6650
 Wire Wire Line
-	6850 3800 6850 5100
-Wire Wire Line
-	6550 5100 6550 3650
+	6850 3800 6850 5150
+Wire Wire Line
+	6550 3650 6550 5150
 Wire Wire Line
 	6550 3650 7250 3650
@@
 NoConn ~ 3650 3450
 NoConn ~ 4400 2700
+Wire Wire Line
+	3900 4250 2900 4250
+NoConn ~ 3850 3450
+Wire Wire Line
+	4200 5800 4200 5850
+Wire Wire Line
+	4200 5450 4200 5500
+Wire Wire Line
+	6550 5450 6550 5500
+Wire Wire Line
+	6850 5500 6850 5450
 $Comp
 L PWR_FLAG #FLG052
 U 1 1 57AB052A
-P 1150 7150
-F 0 "#FLG052" H 1150 7245 50  0001 C CNN
-F 1 "PWR_FLAG" H 1150 7330 50  0000 C CNN
-F 2 "" H 1150 7150 60  0000 C CNN
-F 3 "" H 1150 7150 60  0000 C CNN
-	1    1150 7150
+P 650 6850
+F 0 "#FLG052" H 650 6945 50  0001 C CNN
+F 1 "PWR_FLAG" H 650 7030 50  0000 C CNN
+F 2 "" H 650 6850 60  0000 C CNN
+F 3 "" H 650 6850 60  0000 C CNN
+	1    650  6850
+	-1   0    0    1
+$EndComp
+Wire Wire Line
+	650  6850 650  6800
+Wire Wire Line
+	650  6800 800  6800
+Wire Wire Line
+	800  6725 800  6825
+Connection ~ 800  6800
+NoConn ~ 1000 7125
+Wire Wire Line
+	1400 7125 1400 7325
+Wire Wire Line
+	1400 7325 1375 7325
+$Comp
+L PWR_FLAG #FLG053
+U 1 1 5B3613CB
+P 1400 7250
+F 0 "#FLG053" H 1400 7345 50  0001 C CNN
+F 1 "PWR_FLAG" H 1400 7430 50  0000 C CNN
+F 2 "" H 1400 7250 60  0000 C CNN
+F 3 "" H 1400 7250 60  0000 C CNN
+	1    1400 7250
 	0    1    1    0
 $EndComp
-Wire Wire Line
-	3900 4250 2900 4250
+Connection ~ 1400 7250
 $EndSCHEMATC

Commit message: Ground crystal case
Parts:
- X1: symbol CRYSTAL_SMD -> Crystal_GND2
Connections:
- wire segments 92 -> 94
- no-connect marks 17 -> 15
Changed lines of the file:
@@
 Connection ~ 3550 3650
 $Comp
-L CRYSTAL_SMD X1
+L Crystal_GND2 X1
 U 1 1 572B9603
 P 3750 3450
 F 0 "X1" H 3650 3600 50  0000 C CNN
-F 1 "TSX-3225  X1E0000210013" H 3250 3700 50  0000 L CNN
+F 1 "TSX-3225  X1E0000210013" V 3600 2325 50  0000 L CNN
 F 2 "Crystals:crystal_FA238-TSX3225" H 3750 3450 60  0001 C CNN
 F 3 "" H 3750 3450 60  0000 C CNN
 	1    3750 3450
-	0    1    1    0
+	0    -1   1    0
 $EndComp
-NoConn ~ 3650 3450
 NoConn ~ 4400 2700
 Wire Wire Line
 	3900 4250 2900 4250
-NoConn ~ 3850 3450
 Wire Wire Line
 	4200 5800 4200 5850
@@
 $EndComp
 Connection ~ 1400 7250
+Wire Wire Line
+	3750 3250 3750 3300
+Wire Wire Line
+	3750 3600 3750 3650
+$Comp
+L GND #PWR?
+U 1 1 5B3542B9
+P 3950 3450
+F 0 "#PWR?" H 3950 3200 50  0001 C CNN
+F 1 "GND" H 3950 3300 50  0000 C CNN
+F 2 "" H 3950 3450 60  0000 C CNN
+F 3 "" H 3950 3450 60  0000 C CNN
+	1    3950 3450
+	0    -1   -1   0
+$EndComp
 $EndSCHEMATC

Commit message: Correct pin headers to odd-even
Parts:
- P5: symbol Conn_02x03_Counter_Clockwise -> Conn_02x03_Odd_Even
- X1: symbol Crystal_GND2 -> Crystal_GND3
Changed lines of the file:
@@
 5V
 $Comp
-L Conn_02x03_Counter_Clockwise P5
+L Conn_02x03_Odd_Even P5
 U 1 1 56BA568C
 P 2350 6750
@@
 Connection ~ 3550 3650
 $Comp
-L Crystal_GND2 X1
+L Crystal_GND3 X1
 U 1 1 572B9603
 P 3750 3450

Commit message: Produce BOM with "Boms away"
Parts:
- C28, C29, C30, C31, C32, C33, C34, R20, R21, R22, R23, R_Ser1, R_Ser2: MFR (none) -> -; MPN (none) -> -; SPN (none) -> -; SPR (none) -> -; SPURL (none) -> -
- IC1: MFR (none) -> Microchip Technology; MPN (none) -> ATMEGA328P-AN; SPN (none) -> 131-0270; SPR (none) -> RS; SPURL (none) -> -
- ICSP1: renamed from P5; value ICSP -> HEADER; footprint Pin_Headers:Pin_Header_Straight_2x03 -> Pin_Headers:Pin_Header_Straight_2x03_Pitch2.54mm; MFR (none) -> Harwin; MPN (none) -> M20-9980346; SPN (none) -> 745-7046; SPR (none) -> RS; SPURL (none) -> -
- P4: MFR (none) -> Molex; MPN (none) -> 47590-0001; SPN (none) -> 702-5481; SPR (none) -> RS; SPURL (none) -> -
- RX1: renamed from D4; value RX -> LED; MFR (none) -> Bivar; MPN (none) -> SM0805HC; SPN (none) -> 147-9844; SPR (none) -> RS; SPURL (none) -> -
- SCLK1: renamed from D5; value SCLK -> LED; MFR (none) -> Bivar; MPN (none) -> SM0805HC; SPN (none) -> 147-9844; SPR (none) -> RS; SPURL (none) -> -
- TX1: renamed from D3; value TX -> LED; MFR (none) -> Bivar; MPN (none) -> SM0805HC; SPN (none) -> 147-9844; SPR (none) -> RS; SPURL (none) -> -
- U11: MFR (none) -> TI; MPN (none) -> ISO7242CDW; SPN (none) -> 121-9145; SPR (none) -> RS; SPURL (none) -> -
- U12: MFR (none) -> FTDI Chip; MPN (none) -> FT232RL; SPN (none) -> 406-580; SPR (none) -> RS; SPURL (none) -> -
- X1: value TSX-3225 X1E0000210013 -> TSX-3225 X1E0000210013; MFR (none) -> Epson; MPN (none) -> X1E000021001311; SPN (none) -> 667-6151; SPR (none) -> RS; SPURL (none) -> -

Commit message: BOM corrections (thanks Sean!)
Parts:
- RX1, SCLK1, TX1: SPN 147-9844 -> 174-9844
Changed lines of the file:
@@
 F 5 "SM0805HC" H 0 0 50 0001 C CNN "MPN"
 F 6 "RS" H 0 0 50 0001 C CNN "SPR"
-F 7 "147-9844" H 0 0 50 0001 C CNN "SPN"
+F 7 "174-9844" H 0 0 50 0001 C CNN "SPN"
 F 8 "-" H 0 0 50 0001 C CNN "SPURL"
 	1    4200 5650
@@
 F 5 "SM0805HC" H 0 0 50 0001 C CNN "MPN"
 F 6 "RS" H 0 0 50 0001 C CNN "SPR"
-F 7 "147-9844" H 0 0 50 0001 C CNN "SPN"
+F 7 "174-9844" H 0 0 50 0001 C CNN "SPN"
 F 8 "-" H 0 0 50 0001 C CNN "SPURL"
 	1    6550 5300
@@
 F 5 "SM0805HC" H 0 0 50 0001 C CNN "MPN"
 F 6 "RS" H 0 0 50 0001 C CNN "SPR"
-F 7 "147-9844" H 0 0 50 0001 C CNN "SPN"
+F 7 "174-9844" H 0 0 50 0001 C CNN "SPN"
 F 8 "-" H 0 0 50 0001 C CNN "SPURL"
 	1    6850 5300
