File: PCB/GP22_Power.sch (KiCad schematic (older format))
At the start: 7 parts, among them U10 XC6206

Commit message: Produce BOM with "Boms away"
Parts:
- C21, C22, C23, R35, R36, R37: MFR (none) -> -; MPN (none) -> -; SPN (none) -> -; SPR (none) -> -; SPURL (none) -> -
- U10: MFR (none) -> Torex; MPN (none) -> XC6206P332PR; SPN (none) -> 8796998; SPR (none) -> Farnell; SPURL (none) -> -
