File: PCB/GP22_board.sch (KiCad schematic (older format))
At the start: 53 parts, among them CON1 5V power input, P1 TTLOut1, P13 TTLOut2, P14 TTLOut3, P15 PWR_SEL, P16 FILT_SEL, P2 SineInput, P3 TTLInput, P6 STInput, SW1 START, SW2 STOP1, SW3 STOP2, U2 GP22, U3 LTC6957-4, U4 ISO3088, U5 IDT49FCT, U6 LD1117S33TR, Y1 4MHz, Y2 32.768 kHz

Commit message: Update sch for new kicad version
Parts:
- CON1: symbol BARREL_JACK -> Barrel_Jack
- JP1: symbol JUMPER3 -> Jumper_NC_Dual
- P1, P13, P14, P2, P3, P6: symbol BNC -> Conn_Coaxial
- P15: symbol CONN_01X03 -> Conn_01x03
- P16: symbol CONN_02X02 -> Conn_02x02_Counter_Clockwise
- U6: symbol LD1117S33TR -> LD1117S33TR_SOT223-RESCUE-GP22_board
Connections:
- wire segments 117 -> 121
Changed lines of the file:
@@
 EESchema Schematic File Version 2
+LIBS:GP22_board-rescue
 LIBS:power
 LIBS:device
@@
 $EndComp
 $Comp
-L JUMPER3 JP1
+L Jumper_NC_Dual JP1
 U 1 1 582FEE26
 P 9450 2100
@@
 $EndComp
 $Comp
-L BNC P2
+L Conn_Coaxial P2
 U 1 1 5895BE53
 P 1050 2750
@@
 $EndComp
 $Comp
-L BNC P3
+L Conn_Coaxial P3
 U 1 1 589C34DE
 P 1050 5200
@@
 $EndComp
 $Comp
-L BNC P6
+L Conn_Coaxial P6
 U 1 1 589E7C0D
 P 1125 7050
@@
 GP22_FIRE_UP
 $Comp
-L BNC P1
+L Conn_Coaxial P1
 U 1 1 58B51588
 P 1900 14125
@@
 $EndComp
 $Comp
-L BNC P13
+L Conn_Coaxial P13
 U 1 1 58B597D4
 P 1900 14775
@@
 $EndComp
 $Comp
-L BNC P14
+L Conn_Coaxial P14
 U 1 1 58B59A9A
 P 1900 15400
@@
 $EndComp
 $Comp
-L BARREL_JACK CON1
+L Barrel_Jack CON1
 U 1 1 58B8046C
 P 10325 1225
@@
 $EndComp
 $Comp
-L LD1117S33TR U6
+L LD1117S33TR_SOT223-RESCUE-GP22_board U6
 U 1 1 58B80D8C
-P 7700 1425
-F 0 "U6" H 7700 1675 50  0000 C CNN
-F 1 "LD1117S33TR" H 7700 1625 50  0000 C CNN
-F 2 "TO_SOT_Packages_SMD:SOT-223" H 7700 1525 50  0001 C CNN
-F 3 "" H 7700 1425 50  0000 C CNN
-	1    7700 1425
+P 7700 1375
+F 0 "U6" H 7700 1625 50  0000 C CNN
+F 1 "LD1117S33TR" H 7700 1575 50  0000 C CNN
+F 2 "TO_SOT_Packages_SMD:SOT-223" H 7700 1475 50  0001 C CNN
+F 3 "" H 7700 1375 50  0000 C CNN
+	1    7700 1375
 	-1   0    0    -1
 $EndComp
 $Comp
-L CONN_01X03 P15
+L Conn_01x03 P15
 U 1 1 58B8306A
 P 8775 875
@@
 $EndComp
 $Comp
-L PWR_FLAG #FLG042
-U 1 1 58DFB7EB
-P 8775 1225
-F 0 "#FLG042" H 8775 1320 50  0001 C CNN
-F 1 "PWR_FLAG" H 8775 1405 50  0000 C CNN
-F 2 "" H 8775 1225 50  0000 C CNN
-F 3 "" H 8775 1225 50  0000 C CNN
-	1    8775 1225
-	-1   0    0    1
-$EndComp
-$Comp
-L +3V3 #PWR043
+L +3V3 #PWR042
 U 1 1 58BC7410
 P 6875 9775
-F 0 "#PWR043" H 6875 9625 50  0001 C CNN
+F 0 "#PWR042" H 6875 9625 50  0001 C CNN
 F 1 "+3V3" H 6875 9915 50  0000 C CNN
 F 2 "" H 6875 9775 50  0000 C CNN
@@
 $EndComp
 $Comp
-L CONN_02X02 P16
+L Conn_02x02_Counter_Clockwise P16
 U 1 1 58E19BCD
-P 4350 1700
-F 0 "P16" H 4350 1850 50  0000 C CNN
-F 1 "FILT_SEL" H 4350 1550 50  0000 C CNN
-F 2 "Pin_Headers:Pin_Header_Straight_2x02_Pitch2.54mm" H 4350 500 50  0001 C CNN
-F 3 "" H 4350 500 50  0000 C CNN
-	1    4350 1700
+P 4300 1650
+F 0 "P16" H 4300 1800 50  0000 C CNN
+F 1 "FILT_SEL" H 4300 1500 50  0000 C CNN
+F 2 "Pin_Headers:Pin_Header_Straight_2x02_Pitch2.54mm" H 4300 450 50  0001 C CNN
+F 3 "" H 4300 450 50  0000 C CNN
+	1    4300 1650
 	0    -1   1    0
 $EndComp
 $Comp
-L GND #PWR044
+L GND #PWR043
 U 1 1 58E1A4A6
 P 4350 1350
-F 0 "#PWR044" H 4350 1100 50  0001 C CNN
+F 0 "#PWR043" H 4350 1100 50  0001 C CNN
 F 1 "GND" H 4350 1200 50  0000 C CNN
 F 2 "" H 4350 1350 50  0000 C CNN
@@
 GP22_VCC
 $Comp
-L GND #PWR045
+L GND #PWR044
 U 1 1 58E37A8B
 P 7725 10150
-F 0 "#PWR045" H 7725 9900 50  0001 C CNN
+F 0 "#PWR044" H 7725 9900 50  0001 C CNN
 F 1 "GND" H 7725 10000 50  0000 C CNN
 F 2 "" H 7725 10150 50  0000 C CNN
@@
 	8100 1225 8100 1375
 Connection ~ 9675 1325
-Connection ~ 8775 1225
 Wire Wire Line
 	3800 2300 3800 1750
@@
 $EndComp
 $Comp
-L GND #PWR046
+L GND #PWR045
 U 1 1 58E53605
 P 2575 9950
-F 0 "#PWR046" H 2575 9700 50  0001 C CNN
+F 0 "#PWR045" H 2575 9700 50  0001 C CNN
 F 1 "GND" H 2575 9800 50  0000 C CNN
 F 2 "" H 2575 9950 50  0000 C CNN
@@
 $EndComp
 $Comp
-L GND #PWR047
+L GND #PWR046
 U 1 1 58E6CF97
 P 2600 11175
-F 0 "#PWR047" H 2600 10925 50  0001 C CNN
+F 0 "#PWR046" H 2600 10925 50  0001 C CNN
 F 1 "GND" H 2600 11025 50  0000 C CNN
 F 2 "" H 2600 11175 50  0000 C CNN
@@
 $EndComp
 $Comp
-L GND #PWR048
+L GND #PWR047
 U 1 1 58E72385
 P 2600 12300
-F 0 "#PWR048" H 2600 12050 50  0001 C CNN
+F 0 "#PWR047" H 2600 12050 50  0001 C CNN
 F 1 "GND" H 2600 12150 50  0000 C CNN
 F 2 "" H 2600 12300 50  0000 C CNN
@@
 Text Label 5125 12575 2    60   ~ 0
 GP22_VIO
+Wire Wire Line
+	7300 1375 7400 1375
+Wire Wire Line
+	8100 1375 8000 1375
+Wire Wire Line
+	8750 2500 8750 2450
+Wire Wire Line
+	8750 2100 8750 2150
+$Comp
+L PWR_FLAG #FLG048
+U 1 1 5B37A462
+P 8425 1225
+F 0 "#FLG048" H 8425 1320 50  0001 C CNN
+F 1 "PWR_FLAG" H 8425 1405 50  0000 C CNN
+F 2 "" H 8425 1225 50  0000 C CNN
+F 3 "" H 8425 1225 50  0000 C CNN
+	1    8425 1225
+	-1   0    0    1
+$EndComp
+Connection ~ 8425 1225
 $EndSCHEMATC

Commit message: Correct pin headers to odd-even
Parts:
- P16: symbol Conn_02x02_Counter_Clockwise -> Conn_02x02_Odd_Even
Changed lines of the file:
@@
 $EndComp
 $Comp
-L Conn_02x02_Counter_Clockwise P16
+L Conn_02x02_Odd_Even P16
 U 1 1 58E19BCD
 P 4300 1650

Commit message: Fix the Rotary switch schematic file
Parts:
- SW1, SW2, SW3: symbol ROTARY_SWITCH_ALPS_SRBM -> ROTARY_SWITCH_ALPS_SRBM_FIXED
Changed lines of the file:
@@
 NoConn ~ 2300 9150
 $Comp
-L ROTARY_SWITCH_ALPS_SRBM SW1
+L ROTARY_SWITCH_ALPS_SRBM_FIXED SW1
 U 1 1 58E53617
 P 1875 9650
 F 0 "SW1" H 1750 10310 50  0000 C CNN
-F 1 "START" H 1900 9550 50  0000 C CNN
+F 1 "START" H 2025 9900 50  0000 C CNN
 F 2 "Custom:SP3T_switch" H 1650 10210 50  0001 C CNN
 F 3 "" H 1750 10310 50  0001 C CNN
@@
 NoConn ~ 2325 10375
 $Comp
-L ROTARY_SWITCH_ALPS_SRBM SW2
+L ROTARY_SWITCH_ALPS_SRBM_FIXED SW2
 U 1 1 58E6CFA5
 P 1900 10875
@@
 NoConn ~ 2325 11500
 $Comp
-L ROTARY_SWITCH_ALPS_SRBM SW3
+L ROTARY_SWITCH_ALPS_SRBM_FIXED SW3
 U 1 1 58E72393
 P 1900 12000

Commit message: Produce BOM with "Boms away"
Parts:
- removed P15: PWR_SEL, Pin_Headers:Pin_Header_Straight_1x03_Pitch2.54mm, symbol Conn_01x03
- added POWER_SEL1: JMP, Pin_Headers:Pin_Header_Straight_1x03_Pitch2.54mm, symbol Jumper_NC_Dual
- C1, C12, C13, C14, C15, C16, C17, C18, C19, C2, C24, C25, C26, C27, C3, C4, C5, C56, C57, R1, R2, R3, R32, R33, R34, R38, R4, R5, R6, R7, R8, R9: MFR (none) -> -; MPN (none) -> -; SPN (none) -> -; SPR (none) -> -; SPURL (none) -> -
- CON1: MFR (none) -> Switchcraft; MPN (none) -> RAPC712X; SPN (none) -> 878-6787; SPR (none) -> RS; SPURL (none) -> -
- DISABLE_FLASH1: renamed from JP1; value DISABLE FLASH -> JMP; footprint Pin_Headers:Pin_Header_Straight_1x03 -> Pin_Headers:Pin_Header_Straight_1x03_Pitch2.54mm; MFR (none) -> RS Pro; MPN (none) -> 251-8092; SPN (none) -> 251-8092; SPR (none) -> RS; SPURL (none) -> -
- FILT_SEL1: renamed from P16; value FILT_SEL -> HEADER; MFR (none) -> TE Connectivity; MPN (none) -> 826632-2; SPN (none) -> 669-5288; SPR (none) -> RS; SPURL (none) -> -
- POWER1: renamed from D2; value POWER -> LED; MFR (none) -> Bivar; MPN (none) -> SM0805HC; SPN (none) -> 147-9844; SPR (none) -> RS; SPURL (none) -> -
- START1: renamed from SW1; value START -> DP3T; footprint Custom:SP3T_switch -> Custom:ALPS_Rotary_SRBM; MFR (none) -> Apls Electric; MPN (none) -> SRBM131400; SPN (none) -> 123-9600; SPR (none) -> RS; SPURL (none) -> -
- STInput1: renamed from P6; value STInput -> MMCX; MFR (none) -> Molex; MPN (none) -> 73415-1001; SPN (none) -> 759-5300; SPR (none) -> RS; SPURL (none) -> -
- STOP1: renamed from SW2; value STOP1 -> DP3T; footprint Custom:SP3T_switch -> Custom:ALPS_Rotary_SRBM; MFR (none) -> Apls Electric; MPN (none) -> SRBM131400; SPN (none) -> 123-9600; SPR (none) -> RS; SPURL (none) -> -
- STOP2: renamed from SW3; value STOP2 -> DP3T; footprint Custom:SP3T_switch -> Custom:ALPS_Rotary_SRBM; MFR (none) -> Apls Electric; MPN (none) -> SRBM131400; SPN (none) -> 123-9600; SPR (none) -> RS; SPURL (none) -> -
- SineInput1: renamed from P2; value SineInput -> MMCX; MFR (none) -> Molex; MPN (none) -> 73415-1001; SPN (none) -> 759-5300; SPR (none) -> RS; SPURL (none) -> -
- TTLInput1: renamed from P3; value TTLInput -> MMCX; MFR (none) -> Molex; MPN (none) -> 73415-1001; SPN (none) -> 759-5300; SPR (none) -> RS; SPURL (none) -> -
- TTLOut1: renamed from P1; value TTLOut1 -> MMCX; MFR (none) -> Molex; MPN (none) -> 73415-1001; SPN (none) -> 759-5300; SPR (none) -> RS; SPURL (none) -> -
- TTLOut2: renamed from P13; value TTLOut2 -> MMCX; MFR (none) -> Molex; MPN (none) -> 73415-1001; SPN (none) -> 759-5300; SPR (none) -> RS; SPURL (none) -> -
- TTLOut3: renamed from P14; value TTLOut3 -> MMCX; MFR (none) -> Molex; MPN (none) -> 73415-1001; SPN (none) -> 759-5300; SPR (none) -> RS; SPURL (none) -> -
- U2: MFR (none) -> ACAM; MPN (none) -> TDC-GP22; SPN (none) -> TDC-GP225KT&RCT-ND; SPR (none) -> Digikey; SPURL (none) -> -
- U3: MFR (none) -> Linear; MPN (none) -> LTC6957-4; SPN (none) -> DC1766A-B-ND; SPR (none) -> Digikey; SPURL (none) -> -
- U4: MFR (none) -> TI; MPN (none) -> ISO3088DW; SPN (none) -> 121-9061; SPR (none) -> RS; SPURL (none) -> -
- U5: MFR (none) -> IDT; MPN (none) -> IDT49FCT3805ASOGI; SPN (none) -> 715-4902; SPR (none) -> RS; SPURL (none) -> -
- U6: MFR (none) -> STMicroelectroncs; MPN (none) -> LD1117S33TR; SPN (none) -> 168-6804; SPR (none) -> RS; SPURL (none) -> -
- Y1: MFR (none) -> Mercury; MPN (none) -> H49-4.000-18-30/50/4085; SPN (none) -> 672-0173; SPR (none) -> RS; SPURL (none) -> -
- Y2: MFR (none) -> Micro Crystal; MPN (none) -> CM7V-T1A 32.768kHz 7pF +/-10ppm TA QC; SPN (none) -> 729-3252; SPR (none) -> RS; SPURL (none) -> -

Commit message: BOM corrections (thanks Sean!)
Parts:
- POWER1: SPN 147-9844 -> 174-9844
- U3: SPN DC1766A-B-ND -> LTC6957IMS-4#PBF-ND
Changed lines of the file:
@@
 F 5 "SM0805HC" H 0 0 50 0001 C CNN "MPN"
 F 6 "RS" H 0 0 50 0001 C CNN "SPR"
-F 7 "147-9844" H 0 0 50 0001 C CNN "SPN"
+F 7 "174-9844" H 0 0 50 0001 C CNN "SPN"
 F 8 "-" H 0 0 50 0001 C CNN "SPURL"
 	1    8750 2300
@@
 F 5 "LTC6957-4" H 0 0 50 0001 C CNN "MPN"
 F 6 "Digikey" H 0 0 50 0001 C CNN "SPR"
-F 7 "DC1766A-B-ND" H 0 0 50 0001 C CNN "SPN"
+F 7 "LTC6957IMS-4#PBF-ND" H 0 0 50 0001 C CNN "SPN"
 F 8 "-" H 0 0 50 0001 C CNN "SPURL"
 	1    5400 2750

Commit message: Print schematic
Other:
- note removed: "Not sure about this capacitance: determine by trial and error!"

Commit message: Get final cap values for BOM order with PCBTrain
Parts:
- C1, C2, C3, C5: value C -> 3p3
- C15, C16, C17: value 10p -> x
- R5: value R -> 1M
- R6: value R -> x
Changed lines of the file:
@@
 P 3875 10575
 F 0 "C1" H 3900 10675 50  0000 L CNN
-F 1 "C" H 3900 10475 50  0000 L CNN
+F 1 "3p3" H 3900 10475 50  0000 L CNN
 F 2 "Capacitors_SMD:C_0805_HandSoldering" H 3913 10425 50  0001 C CNN
 F 3 "" H 3875 10575 50  0000 C CNN
@@
 P 3875 11175
 F 0 "C2" H 3900 11275 50  0000 L CNN
-F 1 "C" H 3900 11075 50  0000 L CNN
+F 1 "3p3" H 3900 11075 50  0000 L CNN
 F 2 "Capacitors_SMD:C_0805_HandSoldering" H 3913 11025 50  0001 C CNN
 F 3 "" H 3875 11175 50  0000 C CNN
@@
 P 4275 10875
 F 0 "R5" V 4355 10875 50  0000 C CNN
-F 1 "R" V 4275 10875 50  0000 C CNN
+F 1 "1M" V 4275 10875 50  0000 C CNN
 F 2 "Resistors_SMD:R_0805_HandSoldering" V 4205 10875 50  0001 C CNN
 F 3 "" H 4275 10875 50  0000 C CNN
@@
 P 6975 13125
 F 0 "C5" H 7000 13225 50  0000 L CNN
-F 1 "C" H 7000 13025 50  0000 L CNN
+F 1 "3p3" H 7000 13025 50  0000 L CNN
 F 2 "Capacitors_SMD:C_0805_HandSoldering" H 7013 12975 50  0001 C CNN
 F 3 "" H 6975 13125 50  0000 C CNN
@@
 P 6325 13125
 F 0 "C3" H 6350 13225 50  0000 L CNN
-F 1 "C" H 6350 13025 50  0000 L CNN
+F 1 "3p3" H 6350 13025 50  0000 L CNN
 F 2 "Capacitors_SMD:C_0805_HandSoldering" H 6363 12975 50  0001 C CNN
 F 3 "" H 6325 13125 50  0000 C CNN
@@
 P 6625 12625
 F 0 "R6" V 6705 12625 50  0000 C CNN
-F 1 "R" V 6625 12625 50  0000 C CNN
+F 1 "x" V 6625 12625 50  0000 C CNN
 F 2 "Resistors_SMD:R_0805_HandSoldering" V 6555 12625 50  0001 C CNN
 F 3 "" H 6625 12625 50  0000 C CNN
@@
 P 2575 9850
 F 0 "C15" H 2585 9920 50  0000 L CNN
-F 1 "10p" H 2585 9770 50  0000 L CNN
+F 1 "x" H 2585 9770 50  0000 L CNN
 F 2 "Capacitors_SMD:C_0805_HandSoldering" H 2575 9850 50  0001 C CNN
 F 3 "" H 2575 9850 50  0000 C CNN
@@
 P 2600 11075
 F 0 "C16" H 2610 11145 50  0000 L CNN
-F 1 "10p" H 2610 10995 50  0000 L CNN
+F 1 "x" H 2610 10995 50  0000 L CNN
 F 2 "Capacitors_SMD:C_0805_HandSoldering" H 2600 11075 50  0001 C CNN
 F 3 "" H 2600 11075 50  0000 C CNN
@@
 P 2600 12200
 F 0 "C17" H 2610 12270 50  0000 L CNN
-F 1 "10p" H 2610 12120 50  0000 L CNN
+F 1 "x" H 2610 12120 50  0000 L CNN
 F 2 "Capacitors_SMD:C_0805_HandSoldering" H 2600 12200 50  0001 C CNN
 F 3 "" H 2600 12200 50  0000 C CNN
