File: PCB/InputCoupling.sch (KiCad schematic (older format))
At the start: 11 parts, among them P7 S+ DC/AC, P8 S- DC/AC

Commit message: Update sch for new kicad version
Parts:
- P7, P8: symbol CONN_02X02 -> Conn_02x02_Counter_Clockwise
Changed lines of the file:
@@
 EESchema Schematic File Version 2
+LIBS:GP22_board-rescue
 LIBS:power
 LIBS:device
@@
 AR Path="/589C38E1/5898F4B0" Ref="R19"  Part="1"
 AR Path="/589E6F10/5898F4B0" Ref="R29"  Part="1"
-F 0 "R29" V 6730 3750 50  0000 C CNN
+F 0 "R13" V 6730 3750 50  0000 C CNN
 F 1 "R" V 6650 3750 50  0000 C CNN
 F 2 "Resistors_SMD:R_0805_HandSoldering" V 6580 3750 50  0001 C CNN
@@
 AR Path="/589C38E1/5898F558" Ref="C8"  Part="1"
 AR Path="/589E6F10/5898F558" Ref="C10"  Part="1"
-F 0 "C10" H 6760 3670 50  0000 L CNN
+F 0 "C6" H 6760 3670 50  0000 L CNN
 F 1 "C_Small" V 6800 3250 50  0000 L CNN
 F 2 "Capacitors_SMD:C_0805_HandSoldering" H 6750 3600 50  0001 C CNN
@@
 AR Path="/589C38E1/5898F595" Ref="C9"  Part="1"
 AR Path="/589E6F10/5898F595" Ref="C11"  Part="1"
-F 0 "C11" H 6760 3970 50  0000 L CNN
+F 0 "C7" H 6760 3970 50  0000 L CNN
 F 1 "C_Small" V 6650 3950 50  0000 L CNN
 F 2 "Capacitors_SMD:C_0805_HandSoldering" H 6750 3900 50  0001 C CNN
@@
 AR Path="/589C38E1/5898F62F" Ref="R18"  Part="1"
 AR Path="/589E6F10/5898F62F" Ref="R28"  Part="1"
-F 0 "R28" V 6080 3700 50  0000 C CNN
+F 0 "R12" V 6080 3700 50  0000 C CNN
 F 1 "R" V 6000 3700 50  0000 C CNN
 F 2 "Resistors_SMD:R_0805_HandSoldering" V 5930 3700 50  0001 C CNN
@@
 Connection ~ 6000 4100
 $Comp
-L CONN_02X02 P7
+L Conn_02x02_Counter_Clockwise P7
 U 1 1 5898F928
-P 4750 3350
+P 4700 3300
 AR Path="/5898F23C/5898F928" Ref="P7"  Part="1"
 AR Path="/589C38E1/5898F928" Ref="P9"  Part="1"
 AR Path="/589E6F10/5898F928" Ref="P11"  Part="1"
-F 0 "P11" H 4750 3500 50  0000 C CNN
-F 1 "S+ DC/AC" H 4750 3200 50  0000 C CNN
-F 2 "Pin_Headers:Pin_Header_Straight_2x02_Pitch2.54mm" H 4750 2150 50  0001 C CNN
-F 3 "" H 4750 2150 50  0000 C CNN
-	1    4750 3350
+F 0 "P7" H 4700 3450 50  0000 C CNN
+F 1 "S+ DC/AC" H 4700 3150 50  0000 C CNN
+F 2 "Pin_Headers:Pin_Header_Straight_2x02_Pitch2.54mm" H 4700 2100 50  0001 C CNN
+F 3 "" H 4700 2100 50  0000 C CNN
+	1    4700 3300
 	1    0    0    -1
 $EndComp
@@
 	4500 3275 4500 3400
 $Comp
-L CONN_02X02 P8
+L Conn_02x02_Counter_Clockwise P8
 U 1 1 5898F9B2
-P 4750 4150
+P 4700 4200
 AR Path="/5898F23C/5898F9B2" Ref="P8"  Part="1"
 AR Path="/589C38E1/5898F9B2" Ref="P10"  Part="1"
 AR Path="/589E6F10/5898F9B2" Ref="P12"  Part="1"
-F 0 "P12" H 4750 4300 50  0000 C CNN
-F 1 "S- DC/AC" H 4750 4000 50  0000 C CNN
-F 2 "Pin_Headers:Pin_Header_Straight_2x02_Pitch2.54mm" H 4750 2950 50  0001 C CNN
-F 3 "" H 4750 2950 50  0000 C CNN
-	1    4750 4150
+F 0 "P8" H 4700 4350 50  0000 C CNN
+F 1 "S- DC/AC" H 4700 4050 50  0000 C CNN
+F 2 "Pin_Headers:Pin_Header_Straight_2x02_Pitch2.54mm" H 4700 3000 50  0001 C CNN
+F 3 "" H 4700 3000 50  0000 C CNN
+	1    4700 4200
 	1    0    0    1
 $EndComp
@@
 AR Path="/589C38E1/589D05E6" Ref="R17"  Part="1"
 AR Path="/589E6F10/589D05E6" Ref="R27"  Part="1"
-F 0 "R27" H 7030 3220 50  0000 L CNN
+F 0 "R11" H 7030 3220 50  0000 L CNN
 F 1 "10k" H 7030 3160 50  0000 L CNN
 F 2 "Resistors_SMD:R_0805_HandSoldering" H 7000 3200 50  0001 C CNN
@@
 AR Path="/589C38E1/589D066C" Ref="R16"  Part="1"
 AR Path="/589E6F10/589D066C" Ref="R26"  Part="1"
-F 0 "R26" H 6880 3220 50  0000 L CNN
+F 0 "R10" H 6880 3220 50  0000 L CNN
 F 1 "10k" H 6880 3160 50  0000 L CNN
 F 2 "Resistors_SMD:R_0805_HandSoldering" H 6850 3200 50  0001 C CNN
@@
 AR Path="/589C38E1/589D0720" Ref="R25"  Part="1"
 AR Path="/589E6F10/589D0720" Ref="R31"  Part="1"
-F 0 "R31" H 7155 4220 50  0000 L CNN
+F 0 "R15" H 7155 4220 50  0000 L CNN
 F 1 "10k" H 7155 4160 50  0000 L CNN
 F 2 "Resistors_SMD:R_0805_HandSoldering" H 7125 4200 50  0001 C CNN
@@
 AR Path="/589C38E1/589D0771" Ref="R24"  Part="1"
 AR Path="/589E6F10/589D0771" Ref="R30"  Part="1"
-F 0 "R30" H 6955 4220 50  0000 L CNN
+F 0 "R14" H 6955 4220 50  0000 L CNN
 F 1 "10k" H 6955 4160 50  0000 L CNN
 F 2 "Resistors_SMD:R_0805_HandSoldering" H 6925 4200 50  0001 C CNN
@@
 $EndComp
 $Comp
-L GND #PWR055
+L GND #PWR056
 U 1 1 589D07ED
 P 6850 3100
-AR Path="/5898F23C/589D07ED" Ref="#PWR055"  Part="1"
-AR Path="/589C38E1/589D07ED" Ref="#PWR060"  Part="1"
-AR Path="/589E6F10/589D07ED" Ref="#PWR083"  Part="1"
-F 0 "#PWR083" H 6850 2850 50  0001 C CNN
+AR Path="/5898F23C/589D07ED" Ref="#PWR056"  Part="1"
+AR Path="/589C38E1/589D07ED" Ref="#PWR061"  Part="1"
+AR Path="/589E6F10/589D07ED" Ref="#PWR084"  Part="1"
+F 0 "#PWR084" H 6850 2850 50  0001 C CNN
 F 1 "GND" H 6850 2950 50  0000 C CNN
 F 2 "" H 6850 3100 50  0000 C CNN
@@
 Connection ~ 7125 4100
 $Comp
-L GND #PWR056
+L GND #PWR057
 U 1 1 589D0825
 P 6925 4300
-AR Path="/5898F23C/589D0825" Ref="#PWR056"  Part="1"
-AR Path="/589C38E1/589D0825" Ref="#PWR061"  Part="1"
-AR Path="/589E6F10/589D0825" Ref="#PWR084"  Part="1"
-F 0 "#PWR084" H 6925 4050 50  0001 C CNN
+AR Path="/5898F23C/589D0825" Ref="#PWR057"  Part="1"
+AR Path="/589C38E1/589D0825" Ref="#PWR062"  Part="1"
+AR Path="/589E6F10/589D0825" Ref="#PWR085"  Part="1"
+F 0 "#PWR085" H 6925 4050 50  0001 C CNN
 F 1 "GND" H 6925 4150 50  0000 C CNN
 F 2 "" H 6925 4300 50  0000 C CNN
@@
 N.B. the terminating 50 ohm resistors should not be connected for the "Straight through" option\n\nThe pull up / down resistors are optional and should be connected or not as required. \nFor the ground end of the signal, these resistors will only ever be required if the signal is treated differentially\n(e.g. as by the LTC6957)
 $Comp
-L +3V3 #PWR057
+L +3V3 #PWR058
 U 1 1 58BB05B7
 P 7000 3100
-AR Path="/5898F23C/58BB05B7" Ref="#PWR057"  Part="1"
-AR Path="/589C38E1/58BB05B7" Ref="#PWR062"  Part="1"
-AR Path="/589E6F10/58BB05B7" Ref="#PWR085"  Part="1"
-F 0 "#PWR085" H 7000 2950 50  0001 C CNN
+AR Path="/5898F23C/58BB05B7" Ref="#PWR058"  Part="1"
+AR Path="/589C38E1/58BB05B7" Ref="#PWR063"  Part="1"
+AR Path="/589E6F10/58BB05B7" Ref="#PWR086"  Part="1"
+F 0 "#PWR086" H 7000 2950 50  0001 C CNN
 F 1 "+3V3" H 7000 3240 50  0000 C CNN
 F 2 "" H 7000 3100 50  0000 C CNN
@@
 $EndComp
 $Comp
-L +3V3 #PWR058
+L +3V3 #PWR059
 U 1 1 58BB05EA
 P 7125 4300
-AR Path="/5898F23C/58BB05EA" Ref="#PWR058"  Part="1"
-AR Path="/589C38E1/58BB05EA" Ref="#PWR063"  Part="1"
-AR Path="/589E6F10/58BB05EA" Ref="#PWR086"  Part="1"
-F 0 "#PWR086" H 7125 4150 50  0001 C CNN
+AR Path="/5898F23C/58BB05EA" Ref="#PWR059"  Part="1"
+AR Path="/589C38E1/58BB05EA" Ref="#PWR064"  Part="1"
+AR Path="/589E6F10/58BB05EA" Ref="#PWR087"  Part="1"
+F 0 "#PWR087" H 7125 4150 50  0001 C CNN
 F 1 "+3V3" H 7125 4440 50  0000 C CNN
 F 2 "" H 7125 4300 50  0000 C CNN
@@
 AR Path="/589C38E1/58DC66C6" Ref="D6"  Part="1"
 AR Path="/589E6F10/58DC66C6" Ref="D7"  Part="1"
-F 0 "D7" H 4050 3900 50  0000 C CNN
+F 0 "D1" H 4050 3900 50  0000 C CNN
 F 1 "ESDA5V3SC6" H 3900 4050 50  0000 C CNN
 F 2 "TO_SOT_Packages_SMD:SOT-23-5_HandSoldering" H 3750 3800 50  0001 C CNN
@@
 NoConn ~ 4050 3400
 $Comp
-L GND #PWR059
+L GND #PWR060
 U 1 1 58DC695B
 P 3900 3450
-AR Path="/5898F23C/58DC695B" Ref="#PWR059"  Part="1"
-AR Path="/589C38E1/58DC695B" Ref="#PWR064"  Part="1"
-AR Path="/589E6F10/58DC695B" Ref="#PWR087"  Part="1"
-F 0 "#PWR087" H 3900 3200 50  0001 C CNN
+AR Path="/5898F23C/58DC695B" Ref="#PWR060"  Part="1"
+AR Path="/589C38E1/58DC695B" Ref="#PWR065"  Part="1"
+AR Path="/589E6F10/58DC695B" Ref="#PWR088"  Part="1"
+F 0 "#PWR088" H 3900 3200 50  0001 C CNN
 F 1 "GND" H 3900 3300 50  0000 C CNN
 F 2 "" H 3900 3450 50  0000 C CNN

Commit message: Correct input coupling orientation
Parts:
- P7, P8: symbol Conn_02x02_Counter_Clockwise -> Conn_02x02_Odd_Even
Changed lines of the file:
@@
 Connection ~ 6000 4100
 $Comp
-L Conn_02x02_Counter_Clockwise P7
+L Conn_02x02_Odd_Even P7
 U 1 1 5898F928
 P 4700 3300
@@
 	4500 3275 4500 3400
 $Comp
-L Conn_02x02_Counter_Clockwise P8
+L Conn_02x02_Odd_Even P8
 U 1 1 5898F9B2
 P 4700 4200
@@
 $EndComp
 $Comp
-L GND #PWR056
+L GND #PWR057
 U 1 1 589D07ED
 P 6850 3100
-AR Path="/5898F23C/589D07ED" Ref="#PWR056"  Part="1"
-AR Path="/589C38E1/589D07ED" Ref="#PWR061"  Part="1"
-AR Path="/589E6F10/589D07ED" Ref="#PWR084"  Part="1"
-F 0 "#PWR084" H 6850 2850 50  0001 C CNN
+AR Path="/5898F23C/589D07ED" Ref="#PWR057"  Part="1"
+AR Path="/589C38E1/589D07ED" Ref="#PWR062"  Part="1"
+AR Path="/589E6F10/589D07ED" Ref="#PWR085"  Part="1"
+F 0 "#PWR057" H 6850 2850 50  0001 C CNN
 F 1 "GND" H 6850 2950 50  0000 C CNN
 F 2 "" H 6850 3100 50  0000 C CNN
@@
 Connection ~ 7125 4100
 $Comp
-L GND #PWR057
+L GND #PWR058
 U 1 1 589D0825
 P 6925 4300
-AR Path="/5898F23C/589D0825" Ref="#PWR057"  Part="1"
-AR Path="/589C38E1/589D0825" Ref="#PWR062"  Part="1"
-AR Path="/589E6F10/589D0825" Ref="#PWR085"  Part="1"
-F 0 "#PWR085" H 6925 4050 50  0001 C CNN
+AR Path="/5898F23C/589D0825" Ref="#PWR058"  Part="1"
+AR Path="/589C38E1/589D0825" Ref="#PWR063"  Part="1"
+AR Path="/589E6F10/589D0825" Ref="#PWR086"  Part="1"
+F 0 "#PWR058" H 6925 4050 50  0001 C CNN
 F 1 "GND" H 6925 4150 50  0000 C CNN
 F 2 "" H 6925 4300 50  0000 C CNN
@@
 N.B. the terminating 50 ohm resistors should not be connected for the "Straight through" option\n\nThe pull up / down resistors are optional and should be connected or not as required. \nFor the ground end of the signal, these resistors will only ever be required if the signal is treated differentially\n(e.g. as by the LTC6957)
 $Comp
-L +3V3 #PWR058
+L +3V3 #PWR059
 U 1 1 58BB05B7
 P 7000 3100
-AR Path="/5898F23C/58BB05B7" Ref="#PWR058"  Part="1"
-AR Path="/589C38E1/58BB05B7" Ref="#PWR063"  Part="1"
-AR Path="/589E6F10/58BB05B7" Ref="#PWR086"  Part="1"
-F 0 "#PWR086" H 7000 2950 50  0001 C CNN
+AR Path="/5898F23C/58BB05B7" Ref="#PWR059"  Part="1"
+AR Path="/589C38E1/58BB05B7" Ref="#PWR064"  Part="1"
+AR Path="/589E6F10/58BB05B7" Ref="#PWR087"  Part="1"
+F 0 "#PWR059" H 7000 2950 50  0001 C CNN
 F 1 "+3V3" H 7000 3240 50  0000 C CNN
 F 2 "" H 7000 3100 50  0000 C CNN
@@
 $EndComp
 $Comp
-L +3V3 #PWR059
+L +3V3 #PWR060
 U 1 1 58BB05EA
 P 7125 4300
-AR Path="/5898F23C/58BB05EA" Ref="#PWR059"  Part="1"
-AR Path="/589C38E1/58BB05EA" Ref="#PWR064"  Part="1"
-AR Path="/589E6F10/58BB05EA" Ref="#PWR087"  Part="1"
-F 0 "#PWR087" H 7125 4150 50  0001 C CNN
+AR Path="/5898F23C/58BB05EA" Ref="#PWR060"  Part="1"
+AR Path="/589C38E1/58BB05EA" Ref="#PWR065"  Part="1"
+AR Path="/589E6F10/58BB05EA" Ref="#PWR088"  Part="1"
+F 0 "#PWR060" H 7125 4150 50  0001 C CNN
 F 1 "+3V3" H 7125 4440 50  0000 C CNN
 F 2 "" H 7125 4300 50  0000 C CNN
@@
 NoConn ~ 4050 3400
 $Comp
-L GND #PWR060
+L GND #PWR061
 U 1 1 58DC695B
 P 3900 3450
-AR Path="/5898F23C/58DC695B" Ref="#PWR060"  Part="1"
-AR Path="/589C38E1/58DC695B" Ref="#PWR065"  Part="1"
-AR Path="/589E6F10/58DC695B" Ref="#PWR088"  Part="1"
-F 0 "#PWR088" H 3900 3200 50  0001 C CNN
+AR Path="/5898F23C/58DC695B" Ref="#PWR061"  Part="1"
+AR Path="/589C38E1/58DC695B" Ref="#PWR066"  Part="1"
+AR Path="/589E6F10/58DC695B" Ref="#PWR089"  Part="1"
+F 0 "#PWR061" H 3900 3200 50  0001 C CNN
 F 1 "GND" H 3900 3300 50  0000 C CNN
 F 2 "" H 3900 3450 50  0000 C CNN

Commit message: Produce BOM with "Boms away"
Parts:
- C6, C7, R10, R11, R14, R15: MFR (none) -> -; MPN (none) -> -; SPN (none) -> -; SPR (none) -> -; SPURL (none) -> -
- D1: MFR (none) -> STMicroelectronics; MPN (none) -> ESDA5V3SC6; SPN (none) -> 102-6170; SPR (none) -> RS; SPURL (none) -> -
- P7: value S+ DC/AC -> HEADER; MFR (none) -> TE Connectivity; MPN (none) -> 826632-2; SPN (none) -> 669-5288; SPR (none) -> RS; SPURL (none) -> -
- P8: value S- DC/AC -> HEADER; MFR (none) -> TE Connectivity; MPN (none) -> 826632-2; SPN (none) -> 669-5288; SPR (none) -> RS; SPURL (none) -> -
- R12, R13: value R -> 50R; MFR (none) -> -; MPN (none) -> -; SPN (none) -> -; SPR (none) -> -; SPURL (none) -> -

Commit message: BOM corrections (thanks Sean!)
Parts:
- D1: SPN 102-6170 -> 250-000
Changed lines of the file:
@@
 F 5 "ESDA5V3SC6" H 0 0 50 0001 C CNN "MPN"
 F 6 "RS" H 0 0 50 0001 C CNN "SPR"
-F 7 "102-6170" H 0 0 50 0001 C CNN "SPN"
+F 7 "250-000" H 0 0 50 0001 C CNN "SPN"
 F 8 "-" H 0 0 50 0001 C CNN "SPURL"
 	1    4050 3800

Commit message: Get final cap values for BOM order with PCBTrain
Changed lines of the file:
@@
 AR Path="/589C38E1/5898F928" Ref="P9"  Part="1"
 AR Path="/589E6F10/5898F928" Ref="P11"  Part="1"
-F 0 "S+ DC/AC" H 4700 3450 50  0000 C CNN
+F 0 "P11" H 4700 3450 50  0000 C CNN
 F 1 "HEADER" H 4700 3150 50  0000 C CNN
 F 2 "Pin_Headers:Pin_Header_Straight_2x02_Pitch2.54mm" H 4700 2100 50  0001 C CNN
@@
 AR Path="/589C38E1/5898F9B2" Ref="P10"  Part="1"
 AR Path="/589E6F10/5898F9B2" Ref="P12"  Part="1"
-F 0 "S- DC/AC" H 4700 4350 50  0000 C CNN
+F 0 "P12" H 4700 4350 50  0000 C CNN
 F 1 "HEADER" H 4700 4050 50  0000 C CNN
 F 2 "Pin_Headers:Pin_Header_Straight_2x02_Pitch2.54mm" H 4700 3000 50  0001 C CNN
